File: drone_pcb.kicad_pcb (KiCad board)
At the start: 2 copper layers, 52 x 52 mm, 31 parts, among them J1 HappyModel EP1, J2 BATT, M1 Motor_DC, M2 Motor_DC, M3 Motor_DC, M4 Motor_DC, Q1 AO3400A, Q2 AO3400A, Q3 AO3400A, Q4 AO3400A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

Commit message: in the middle of adding traces
Parts:
- removed M1, M2, M3, M4: Motor_DC, Connector_PinHeader_2.00mm:PinHeader_1x02_P2.00mm_Vertical
- added J10: M4_NEG, Connector_Wire:SolderWire-0.25sqmm_1x01_D0.65mm_OD1.7mm, F.Cu at (112.0, 126.5)
- added J3: M1_NEG, Connector_Wire:SolderWire-0.25sqmm_1x01_D0.65mm_OD1.7mm, F.Cu at (64.5, 79.5)
- added J4: M1_POS, Connector_Wire:SolderWire-0.25sqmm_1x01_D0.65mm_OD1.7mm, F.Cu at (64.5, 83.0)
- added J5: M2_POS, Connector_Wire:SolderWire-0.25sqmm_1x01_D0.65mm_OD1.7mm, F.Cu at (112.0, 82.5)
- added J6: M2_NEG, Connector_Wire:SolderWire-0.25sqmm_1x01_D0.65mm_OD1.7mm, F.Cu at (112.0, 79.5)
- added J7: M3_POS, Connector_Wire:SolderWire-0.25sqmm_1x01_D0.65mm_OD1.7mm, F.Cu at (64.0, 123.5)
- added J8: M3_NEG, Connector_Wire:SolderWire-0.25sqmm_1x01_D0.65mm_OD1.7mm, F.Cu at (64.0, 126.5)
- added J9: M4_POS, Connector_Wire:SolderWire-0.25sqmm_1x01_D0.65mm_OD1.7mm, F.Cu at (112.0, 123.5)
- moved D2 80.6 mm to (110.5, 87.2), turned to 180 degrees
- moved D4 78.1 mm to (110.0, 119.5), turned to 180 degrees
- moved Q2 72.8 mm to (107.2, 81.2)
- moved GATE3 70.6 mm to (73.5, 127.0), turned to 180 degrees
- moved Q4 69.9 mm to (107.5, 126.0)
- moved A1 64.8 mm to (88.4, 103.1)
- moved GATE4 62.4 mm to (103.2, 124.5)
- moved PULLDOWN3 57.0 mm to (73.5, 124.8)
- moved J1 55.4 mm to (72.8, 107.5), turned to 180 degrees
- moved PULLDOWN4 53.2 mm to (103.2, 126.8), turned to 180 degrees
- moved C2 48.8 mm to (110.0, 103.0)
- moved GATE2 45.3 mm to (103.2, 80.0)
- moved Q1 36.8 mm to (69.0, 80.5), turned to 180 degrees
- moved D1 36.7 mm to (66.5, 88.5)
- moved D3 34.8 mm to (66.0, 118.0)
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- renumbered GATE3 to GATE2, GATE2 to GATE3, PULLDOWN3 to PULLDOWN2, PULLDOWN2 to PULLDOWN3
Connections:
- A1 pad 10: /M2_PWM -> /M3_PWM
- A1 pad 11: /M3_PWM -> unconnected-(A1-GPIO8-Pad11)
- A1 pad 12: /M4_PWM -> unconnected-(A1-GPIO9-Pad12)
- A1 pad 26: unconnected-(A1-GPIO20-Pad26)_1 -> /M4_PWM
- A1 pad 27: unconnected-(A1-GPIO21-Pad27) -> /M2_PWM
Routing:
- net /PWR: track 0.00 -> 135.5 mm, vias 0 -> 17
- net Net-(J1-VDD): track 0.00 -> 48.8 mm, vias 0 -> 2
- net /M2_PWM: track 0.00 -> 36.2 mm
- net /M3_PWM: track 0.00 -> 28.0 mm
- net /IMU_INT: track 0.00 -> 25.1 mm
- net /M1_PWM: track 0.00 -> 24.8 mm
- net /RC_RX: track 0.00 -> 22.6 mm
- net /RC_TX: track 0.00 -> 21.9 mm
- net /IMU_SDA: track 0.00 -> 19.4 mm
- net GND: track 0.00 -> 19.1 mm, vias 0 -> 14
- net /M4_PWM: track 0.00 -> 14.0 mm
- net /IMU_SCL: track 0.00 -> 13.1 mm
- net Net-(D3-A): track 0.00 -> 12.9 mm, vias 0 -> 2
- net Net-(D1-A): track 0.00 -> 12.5 mm, vias 0 -> 2
- net Net-(D2-A): track 0.00 -> 11.4 mm, vias 0 -> 2
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- added copper zone on In2.Cu, net /PWR
- added copper zone on In1.Cu, net GND
Other:
- board size 52 x 52 mm -> 52.5 x 52.5 mm
- copper layers 2 -> 4

Commit message: first draft (not usable)
Parts:
- moved U1 0.18 mm to (88.4, 103.2)
- moved J10 0.10 mm to (112.1, 126.5)
- moved J9 0.10 mm to (112.1, 123.5)
Routing:
- net GND: track 19.1 -> 27.6 mm, vias 14 -> 16
- net /PWR: track 135.5 -> 132.3 mm
- net Net-(D4-A): track 11.0 -> 12.8 mm
- net /M2_PWM: track 36.2 -> 37.2 mm
Other:
- board text added: "R1"

Commit message: final draft i think
Parts:
- added C3: 2.2nF, Capacitor_SMD:C_0805_2012Metric, F.Cu at (90.2, 99.0)
- added C4: 0.1uF, Capacitor_SMD:C_0805_2012Metric, F.Cu at (92.9, 106.7)
- added C5: 0.1uF, Capacitor_SMD:C_0805_2012Metric, F.Cu at (86.8, 107.6)
- added C6: 0.1uF, Capacitor_SMD:C_0805_2012Metric, F.Cu at (93.0, 103.5)
- added C7: 22uF, Capacitor_SMD:C_0805_2012Metric, F.Cu at (84.4, 116.0)
- added C8: 100µF, Capacitor_SMD:C_1206_3216Metric, F.Cu at (108.1, 105.3)
- added L1: 2.2uH, Inductor_SMD:L_1008_2520Metric, F.Cu at (87.5, 115.2)
- added R3: 4.7kΩ, Resistor_SMD:R_0805_2012Metric, F.Cu at (83.3, 95.8)
- added R4: 4.7kΩ, Resistor_SMD:R_0805_2012Metric, F.Cu at (85.7, 95.8)
- added R6: 910kΩ, Resistor_SMD:R_0805_2012Metric, F.Cu at (91.1, 118.2)
- added R7: 100kΩ, Resistor_SMD:R_0805_2012Metric, F.Cu at (93.6, 118.2)
- added U3: MPU-6050, Sensor_Motion:InvenSense_QFN-24_4x4mm_P0.5mm, F.Cu at (88.4, 102.8)
- C2: value 220µF -> 100µF; footprint Capacitor_SMD:C_1210_3225Metric -> Capacitor_SMD:C_1206_3216Metric
- U1: value OC09600 -> TLV61070ADBV; footprint OC09600:MODULE_OC09600 -> Package_TO_SOT_SMD:SOT-23-6
- moved U1 15.1 mm to (87.6, 118.3)
- moved J1 5.54 mm to (74.0, 112.9)
- moved U2 2.83 mm to (104.6, 90.8)
- moved C_3 2.49 mm to (101.6, 93.8), turned to -90 degrees
- moved C1 2.40 mm to (108.1, 107.7), turned to 180 degrees
- moved R1 1.94 mm to (102.8, 102.3), turned to 180 degrees
- moved C2 1.92 mm to (108.1, 102.7), turned to 180 degrees
- moved D2 1.50 mm to (110.1, 88.7)
- moved R2 1.48 mm to (102.8, 104.3)
- moved Q4 1.29 mm to (107.0, 124.8)
- moved D3 0.94 mm to (66.8, 118.5)
- moved J7 0.94 mm to (64.8, 124.0)
- moved J8 0.89 mm to (64.8, 126.9)
- moved Q3 0.86 mm to (69.7, 125.5)
- moved GATE4 0.81 mm to (102.7, 123.9)
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Connections:
- A1 pad 10: /M3_PWM -> /IMU_SCL
- A1 pad 11: unconnected-(A1-GPIO8-Pad11) -> /RC_RX
- A1 pad 12: unconnected-(A1-GPIO9-Pad12) -> /RC_TX
- A1 pad 16: /RC_RX -> unconnected-(A1-GPIO12-Pad16)_1
- A1 pad 17: /RC_TX -> /M3_PWM
- A1 pad 27: /M2_PWM -> unconnected-(A1-GPIO21-Pad27)
- A1 pad 29: unconnected-(A1-GPIO22-Pad29)_1 -> /IMU_INT
- A1 pad 34: unconnected-(A1-GPIO28_ADC2-Pad34) -> /M2_PWM
- A1 pad 4: /IMU_SDA -> unconnected-(A1-GPIO2-Pad4)_1
- A1 pad 5: /IMU_SCL -> /M1_PWM
- A1 pad 7: /IMU_INT -> unconnected-(A1-GPIO5-Pad7)
- A1 pad 9: /M1_PWM -> /IMU_SDA
- C_3 pad 1: /PWR -> Net-(U1-V_{OUT})
- C_4 pad 1: Net-(J1-VDD) -> /3.3V
- U2 pad 1: /PWR -> Net-(U1-V_{OUT})
- U2 pad 3: /PWR -> Net-(U1-V_{OUT})
- U2 pad 5: Net-(J1-VDD) -> /3.3V
Routing:
- net /PWR: track 132.3 -> 24.6 mm, vias 17 -> 12
- net Net-(J1-VDD): track 48.8 -> 0.00 mm, vias 2 -> 0
- net /M2_PWM: track 37.2 -> 18.9 mm
- net /IMU_INT: track 25.1 -> 8.54 mm
- net /RC_RX: track 22.6 -> 6.52 mm
- net /RC_TX: track 21.9 -> 5.90 mm
- net /M3_PWM: track 28.0 -> 13.2 mm
- net /M1_PWM: track 24.8 -> 10.8 mm
- net Net-(U1-V_{OUT}): track 0.00 -> 11.6 mm, vias 0 -> 5
- net GND: track 27.6 -> 36.4 mm, vias 16 -> 26
- net Net-(U3-VLOGIC): track 0.00 -> 7.29 mm, vias 0 -> 3
- net /3.3V: track 0.00 -> 7.09 mm, vias 0 -> 4
- net /IMU_SDA: track 19.4 -> 12.6 mm, vias 0 -> 2
- net Net-(U1-V_{FB}): track 0.00 -> 5.74 mm
- net Net-(U3-REGOUT): track 0.00 -> 4.41 mm
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- added copper zone on In2.Cu, net /3.3V
- added copper zone on In2.Cu, net Net-(U1-V_{OUT})
- added copper zone on In2.Cu, net Net-(U3-VLOGIC)
Other:
- board text added: "J9"
- board text added: "awesome drone project"

Commit message: actual final draft
Parts:
- added G***: LOGO, images:jokebear_dancing, F.Cu at (69.7, 96.2)
- added G***: LOGO, images:jokebear_sleep, F.Cu at (73.3, 88.0)
- added G***: LOGO, images:chiikawa, F.Cu at (105.5, 113.1)
- added G***: LOGO, images:jokebear, F.Cu at (73.4, 118.2)
- moved A1 0.12 mm to (88.3, 103.1)
Connections:
- C7 pad 1: Net-(U1-V_{OUT}) -> Net-(J1-Pin_2)
- C_3 pad 1: Net-(U1-V_{OUT}) -> Net-(J1-Pin_2)
- J1 pad 2: Net-(J1-VDD) -> Net-(J1-Pin_2)
- R6 pad 1: Net-(U1-V_{OUT}) -> Net-(J1-Pin_2)
- U1 pad 5: Net-(U1-V_{OUT}) -> Net-(J1-Pin_2)
- U2 pad 1: Net-(U1-V_{OUT}) -> Net-(J1-Pin_2)
- U2 pad 3: Net-(U1-V_{OUT}) -> Net-(J1-Pin_2)
Routing:
- net Net-(U1-V_{OUT}): track 11.6 -> 0.00 mm, vias 5 -> 0
- net Net-(J1-Pin_2): track 0.00 -> 11.6 mm, vias 0 -> 5
- net /PWR: track 24.6 -> 22.6 mm, vias 12 -> 11
- net GND: track 36.4 -> 34.5 mm, vias 26 -> 25
- net /M1_PWM: track 10.8 -> 11.8 mm
- added copper zone on In2.Cu, net Net-(J1-Pin_2)
- removed copper zone on In2.Cu, net Net-(U1-V_{OUT})
Other:
- board text added: "drc initially fails b/c i have components in the area of the pico, but on the actual board the pico will be elevated so these are not relevant. i turned off drc check for {dblquote}items not allowed{dblquote}. also antenna area is not relevant b/c i'm not using the wifi version of the pico"
- board text removed: "awesome drone project"
