File: drone_pcb.kicad_sch (KiCad schematic)
At the start: 23 parts, among them J1 HappyModel EP1, J2 MPU-6050, M1 Motor_DC, M2 Motor_DC, M3 Motor_DC, M4 Motor_DC, Q1 AO3400A, Q2 AO3400A, Q3 AO3400A, Q4 AO3400A

Commit message: schematic done now i think???
Parts:
- removed J2: MPU-6050, symbol Connector:Conn_01x08_Pin
- added C1: 100nF, Capacitor_SMD:C_0805_2012Metric, symbol Device:C
- added C2: 220µF, Capacitor_SMD:C_1210_3225Metric, symbol Device:C_Polarized
- added C_3, C_4: 4.7uF, Capacitor_SMD:C_0805_2012Metric, symbol Device:C
- added J2: BATT, Connector_JST:JST_PH_S2B-PH-K_1x02_P2.00mm_Horizontal, symbol Connector_Generic:Conn_01x02
- added R1, R2: 10kΩ, Resistor_SMD:R_0805_2012Metric, symbol Device:R
- added U1: OC09600, OC09600:MODULE_OC09600, symbol OC09600:OC09600
- added U2: AP2112K-3.3, Package_TO_SOT_SMD:SOT-23-5, symbol Regulator_Linear:AP2112K-3.3
- GATE1, GATE2, GATE3, GATE4: renamed from GATE; footprint (none) -> Resistor_SMD:R_0805_2012Metric
- J1: footprint (none) -> Connector_PinHeader_2.54mm:PinHeader_1x04_P2.54mm_Vertical
- M1, M2, M3, M4: footprint (none) -> Connector_PinHeader_2.00mm:PinHeader_1x02_P2.00mm_Vertical
- PULLDOWN1, PULLDOWN2, PULLDOWN3, PULLDOWN4: renamed from PULLDOWN; footprint (none) -> Resistor_SMD:R_0805_2012Metric
Connections:
- net GND: now also C1.2, C2.2, C_3.2, C_4.2, J2.2 (GND), R2.2, U1.AD0, U1.GND, U2.2 (GND)
- net M1_PWM: now also PULLDOWN1.2
- net M2_PWM: now also PULLDOWN3.2
- net M3_PWM: now also PULLDOWN2.2
- net M4_PWM: now also PULLDOWN4.2
- net at GATE2.2, Q3.1 (G): no longer PULLDOWN2.2
- net at GATE4.2, Q4.1 (G): no longer PULLDOWN4.2
- net at GATE1.2, Q1.1 (G): no longer PULLDOWN1.2
- net at GATE3.2, Q2.1 (G): no longer PULLDOWN3.2
- net at J1.2 (VDD): now also C_4.1, U1.VCC, U2.5 (VOUT); no longer A1.36 (3V3)
- net IMU_SCL: now reaches A1.5 (GPIO3)
- net IMU_SCL: now also U1.SCL
- net IMU_SDA: now reaches A1.4 (GPIO2)
- net IMU_SDA: now also U1.SDA
- net RC_RX: now reaches A1.16 (GPIO12), J1.4 (RX)
- net RC_TX: now reaches A1.17 (GPIO13), J1.3 (TX)
- net at A1.31 (GPIO26_ADC0): now also R1.2, R2.1
- net IMU_INT: now reaches A1.7 (GPIO5)
- net IMU_INT: now also U1.INT
- net +3.7V renamed PWR
- net PWR: now also C1.1, C2.1, C_3.1, J2.1 (3.7V), R1.1, U2.1 (VIN), U2.3 (EN)
- no-connect marks 10 -> 24
Other:
- note added: "BATTERY"
- note added: "awesome drone project"
- moved on the sheet: A1, D1, D2, D3, D4, GATE1, GATE2, GATE3, GATE4, J1, M1, M2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

Commit message: in the middle of adding traces
Parts:
- removed M1, M2, M3, M4: Motor_DC, Connector_PinHeader_2.00mm:PinHeader_1x02_P2.00mm_Vertical, symbol Motor:Motor_DC
- added J10: M4_NEG, Connector_Wire:SolderWire-0.25sqmm_1x01_D0.65mm_OD1.7mm, symbol Connector_Generic:Conn_01x01
- added J3: M1_NEG, Connector_Wire:SolderWire-0.25sqmm_1x01_D0.65mm_OD1.7mm, symbol Connector_Generic:Conn_01x01
- added J4: M1_POS, Connector_Wire:SolderWire-0.25sqmm_1x01_D0.65mm_OD1.7mm, symbol Connector_Generic:Conn_01x01
- added J5: M2_POS, Connector_Wire:SolderWire-0.25sqmm_1x01_D0.65mm_OD1.7mm, symbol Connector_Generic:Conn_01x01
- added J6: M2_NEG, Connector_Wire:SolderWire-0.25sqmm_1x01_D0.65mm_OD1.7mm, symbol Connector_Generic:Conn_01x01
- added J7: M3_POS, Connector_Wire:SolderWire-0.25sqmm_1x01_D0.65mm_OD1.7mm, symbol Connector_Generic:Conn_01x01
- added J8: M3_NEG, Connector_Wire:SolderWire-0.25sqmm_1x01_D0.65mm_OD1.7mm, symbol Connector_Generic:Conn_01x01
- added J9: M4_POS, Connector_Wire:SolderWire-0.25sqmm_1x01_D0.65mm_OD1.7mm, symbol Connector_Generic:Conn_01x01
- renumbered GATE3 to GATE2, GATE2 to GATE3, PULLDOWN3 to PULLDOWN2, PULLDOWN2 to PULLDOWN3
Connections:
- net M2_PWM: now also A1.27 (GPIO21); no longer A1.10 (GPIO7)
- net M3_PWM: now also A1.10 (GPIO7); no longer A1.11 (GPIO8)
- net M4_PWM: now also A1.26 (GPIO20); no longer A1.12 (GPIO9)
- net PWR: now also J4.1 (Pin_1), J5.1 (Pin_1), J7.1 (Pin_1), J9.1 (Pin_1)
- net at D3.2 (A), Q3.3 (D): now also J8.1 (Pin_1)
- net at D2.2 (A), Q2.3 (D): now also J6.1 (Pin_1)
- net at D4.2 (A), Q4.3 (D): now also J10.1 (Pin_1)
- net at D1.2 (A), Q1.3 (D): now also J3.1 (Pin_1)
- no-connect marks 24 -> 22
Other:
- moved on the sheet: R1, R2

Commit message: final draft i think
Parts:
- removed J1: HappyModel EP1, Connector_PinHeader_2.54mm:PinHeader_1x04_P2.54mm_Vertical, symbol Connector:Conn_01x04_Pin
- removed U1: OC09600, OC09600:MODULE_OC09600, symbol OC09600:OC09600
- added C3: 2.2nF, Capacitor_SMD:C_0805_2012Metric, symbol Device:C
- added C4, C5, C6: 0.1uF, Capacitor_SMD:C_0805_2012Metric, symbol Device:C
- added C7: 22uF, Capacitor_SMD:C_0805_2012Metric, symbol Device:C
- added C8: 100µF, Capacitor_SMD:C_1206_3216Metric, symbol Device:C_Polarized
- added L1: 2.2uH, Inductor_SMD:L_1008_2520Metric, symbol Device:L
- added R3, R4: 4.7kΩ, Resistor_SMD:R_0805_2012Metric, symbol Device:R
- added R6: 910kΩ, Resistor_SMD:R_0805_2012Metric, symbol Device:R
- added R7: 100kΩ, Resistor_SMD:R_0805_2012Metric, symbol Device:R
- added U1: TLV61070ADBV, Package_TO_SOT_SMD:SOT-23-6, symbol Regulator_Switching:TLV61070ADBV
- added U3: MPU-6050, Sensor_Motion:InvenSense_QFN-24_4x4mm_P0.5mm, symbol Sensor_Motion:MPU-6050
- C2: value 220µF -> 100µF; footprint Capacitor_SMD:C_1210_3225Metric -> Capacitor_SMD:C_1206_3216Metric
Connections:
- net GND: now also C3.2, C4.2, C7.2, C8.2, R7.2, U1.2 (GND), U3.1 (CLKIN), U3.11 (FSYNC), U3.18 (GND), U3.9 (AD0)
- net IMU_INT: now also A1.29 (GPIO22), U3.12 (INT); no longer A1.7 (GPIO5)
- net IMU_SCL: now also A1.10 (GPIO7), R4.2, U3.23 (SCL); no longer A1.5 (GPIO3)
- net IMU_SDA: now also A1.9 (GPIO6), R3.2, U3.24 (SDA); no longer A1.4 (GPIO2)
- net M1_PWM: now also A1.5 (GPIO3); no longer A1.9 (GPIO6)
- net M2_PWM: now also A1.34 (GPIO28_ADC2); no longer A1.27 (GPIO21)
- net M3_PWM: now also A1.17 (GPIO13); no longer A1.10 (GPIO7)
- net PWR: now also C8.1, L1.2, U1.3 (EN), U1.6 (V_{IN}); no longer C_3.1, U2.1 (VIN), U2.3 (EN)
- net RC_RX: now also A1.11 (GPIO8); no longer A1.16 (GPIO12)
- net RC_TX: now also A1.12 (GPIO9); no longer A1.17 (GPIO13)
- net 3.3V: now reaches C_4.1, U2.5 (VOUT)
- net 3.3V: now also C5.1, C6.1
- new net: C4.1, U3.10 (REGOUT)
- new net: L1.1, U1.1 (SW)
- new net: R6.2, R7.1, U1.4 (V_{FB})
- new net: C7.1, C_3.1, R6.1, U1.5 (V_{OUT}), U2.1 (VIN), U2.3 (EN)
- new net: C6.2, U3.13 (VDD)
- new net: C3.1, U3.20 (CPOUT)
- new net: C5.2, R3.1, R4.1, U3.8 (VLOGIC)
- no-connect marks 22 -> 24
Other:
- note added: "MPU-6050 & Pullup Resistors"
- moved on the sheet: A1, C2, C_3, C_4, R1, R2, U2

Commit message: actual final draft
Parts:
- added J1: HappyModel EP1, Connector_PinHeader_2.54mm:PinHeader_1x04_P2.54mm_Vertical, symbol Connector:Conn_01x04_Pin
Connections:
- net GND: now also J1.1 (Pin_1)
- net RC_RX: now also J1.4 (Pin_4)
- net RC_TX: now also J1.3 (Pin_3)
- net at C7.1, C_3.1, R6.1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: now also J1.2 (Pin_2)
Other:
- note added: "U1 outputs 5V, which will definitely power J1. This is just to ensure U2 has more than enough input voltage to work, since 3.7V is near the lower bound."
Changed lines of the file:
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@@
 		)
 	)
+	(text "U1 outputs 5V, which will definitely power J1. \nThis is just to ensure U2 has more than enough \ninput voltage to work, since 3.7V is near the \nlower bound."
+		(exclude_from_sim no)
+		(at 133.604 98.044 0)
+		(effects
+			(font
+				(size 0.762 0.762)
+			)
+		)
+	)
 	(text "awesome drone project"
 		(exclude_from_sim no)
@@
 					(unit 1)
 				)
+			)
+		)
+	)
+	(symbol
+		(lib_id "Connector:Conn_01x04_Pin")
+		(at 137.16 54.61 0)
+		(unit 1)
+		(body_style 1)
+		(exclude_from_sim no)
+		(in_bom yes)
+		(on_board yes)
+		(in_pos_files yes)
+		(dnp no)
+		(fields_autoplaced yes)
+		(property "Reference" "J1"
+			(at 137.795 46.99 0)
+			(show_name no)
+			(do_not_autoplace no)
+			(effects
+				(font
+					(size 1.27 1.27)
+				)
+			)
+		)
+		(property "Value" "HappyModel EP1"
+			(at 137.795 49.53 0)
+			(show_name no)
+			(do_not_autoplace no)
+			(effects
+				(font
+					(size 1.27 1.27)
+				)
+			)
+		)
+		(property "Footprint" "Connector_PinHeader_2.54mm:PinHeader_1x04_P2.54mm_Vertical"
+			(at 137.16 54.61 0)
+			(hide yes)
+			(show_name no)
+			(do_not_autoplace no)
+			(effects
+				(font
+					(size 1.27 1.27)
+				)
+			)
+		)
+		(property "Datasheet" ""
+			(at 137.16 54.61 0)
+			(hide yes)
+			(show_name no)
+			(do_not_autoplace no)
+			(effects
+				(font
+					(size 1.27 1.27)
+				)
+			)
+		)
+		(property "Description" "Generic connector, single row, 01x04, script generated"
+			(at 137.16 54.61 0)
+			(hide yes)
+			(show_name no)
+			(do_not_autoplace no)
+			(effects
+				(font
+					(size 1.27 1.27)
+				)
+			)
+		)
+		(pin "2"
+		)
+		(pin "1"
+		)
+		(pin "3"
+		)
+		(pin "4"
+		)
+		(instances
+			(project "drone_pcb"
+				(path "/83c625e1-a29f-4d99-8503-8e62b4e27419"
+					(reference "J1")
+					(unit 1)
+				)
